File: trinketm0fader_60mm.brd (EAGLE design)
At the start: 52.1 x 76.2 mm, 11 parts, among them IC1 74AHCT1G125DBV

Commit message: cleanup
Parts:
- moved J4 4.14 mm to (12.0, 75.3)
- moved R4 3.89 mm to (6.10, 73.5)
- moved J3 3.03 mm to (20.3, 70.2)
- moved J5 2.54 mm to (25.9, 75.3)
Routing:
- net 2: track 53.4 -> 57.9 mm
- net 2LS: track 17.9 -> 22.0 mm
- net DI: track 29.4 -> 27.0 mm
- net +3V3: track 70.5 -> 72.5 mm
- net 1: track 57.6 -> 59.3 mm
- net N$1: track 14.3 -> 12.7 mm
- net 0: track 41.3 -> 39.8 mm
- net 3: track 80.9 -> 79.3 mm
- net +5V: track 40.1 -> 41.6 mm
Other:
- board size 52.1 x 76.2 mm -> 52.1 x 78.7 mm
- board text added: "- Selectable 3V / 5V LED power 5V via USB 3V provided by TrinketM0 - Selectable 3V / 5V data pin logic 3V = direct from TrinketM0 5V = via level converter"
- board text added: "B"
- board text added: "H"
- board text added: "Keep clear for USB cable"
- board text added: "Neopixel"
- board text added: "S"
- board text added: "Tester"
- board text added: "dV"
- board text added: "data"
- board text added: "github.com/todbot/neopixeltester trinketm0fader_60mm @todbot 12Aug2019"
- board text added: "ledV"
- board text added: "neopixel"
- board text added: "power"
- board text added: "strip"
- board text removed: "DIN"
- board text removed: "LEDV"
- board text removed: "Neopixel Tester"
- board text removed: "neopixel strip"
