File: trinketm0fader_35mmad.brd (EAGLE design)
At the start: 53.3 x 58.4 mm, 11 parts, among them IC1 74AHCT1G125DBV

Commit message: oops
Routing:
- net +3V3: track 66.1 -> 53.7 mm
- net 4: track 59.2 -> 63.3 mm
- net 3: track 70.6 -> 74.0 mm
- net 1: track 44.8 -> 45.4 mm
Other:
- board text added: "0"
- board text added: "1"
- board text added: "2"
- board text added: "3"
- board text added: "4"
- board text added: "R"
- board text added: "trinketm0fader_35mmad @todbot 17Aug2019"
- board text removed: "trinketm0fader_60mm @todbot 12Aug2019"
